File: hardware/kicad/bench-breathe.kicad_sch (KiCad schematic)
At the start: 10 parts, among them J1 USB4105-GF-A, U1 ESP32-C3-WROOM-02-N4, U2 SPS30, U3 SGP40-D-R4, U4 SHT40-AD1B-R2, U5 TPS62162DSGR, U6 TPD4E05U06DQAR, U7 TPS22919DCKR

Commit message: hardware: complete A0 schematic
Parts:
- removed J1: USB4105-GF-A, symbol Connector_Generic:Conn_01x16
- removed U1: ESP32-C3-WROOM-02-N4, symbol Connector_Generic:Conn_01x19
- removed U2: SPS30, symbol Connector_Generic:Conn_01x05
- removed U3: SGP40-D-R4, symbol Connector_Generic:Conn_01x06
- removed U4: SHT40-AD1B-R2, symbol Sensor_Humidity:SHT4x
- removed U5: TPS62162DSGR, symbol Regulator_Switching:TPS62162DSG
- removed U6: TPD4E05U06DQAR, symbol Connector_Generic:Conn_01x10
- removed U7: TPS22919DCKR, symbol Connector_Generic:Conn_01x06
- added C1, C10, C3: 10uF 10V X5R, Capacitor_SMD:C_1206_3216Metric, symbol Device:C
- added C2: 22uF 16V X5R, Capacitor_SMD:C_1206_3216Metric, symbol Device:C
- added C4, C6, C8, C9: 100nF 50V X7R, Capacitor_SMD:C_0603_1608Metric, symbol Device:C
- added C5, C7: 1uF 16V X7R, Capacitor_SMD:C_0603_1608Metric, symbol Device:C
- added D2: GREEN STATUS, LED_SMD:LED_0603_1608Metric, symbol Device:LED
- added J1: USB4105-GF-A, Connector_USB:USB_C_Receptacle_GCT_USB4105-xx-A_16P_TopMnt_Horizontal, symbol bench-breathe:USB4105-GF-A
- added J2: SPS30 HARNESS, Connector_JST:JST_PH_S5B-PH-K_1x05_P2.00mm_Horizontal, symbol Connector_Generic:Conn_01x05
- added J3: DEBUG / PROGRAM 3V3, Connector_PinHeader_2.54mm:PinHeader_1x06_P2.54mm_Vertical, symbol Connector_Generic:Conn_01x06
- added L1: 2.2uH 1.3A, Inductor_SMD:L_1008_2520Metric, symbol Device:L
- added R1, R2: 5.1k 1%, Resistor_SMD:R_0603_1608Metric, symbol Device:R
- added R10, R4, R8: 10k 1%, Resistor_SMD:R_0603_1608Metric, symbol Device:R
- added R11, R12: 0R 1%, Resistor_SMD:R_0603_1608Metric, symbol Device:R
- added R3: 100k 1%, Resistor_SMD:R_0603_1608Metric, symbol Device:R
- added R5, R6: 4.7k 1%, Resistor_SMD:R_0603_1608Metric, symbol Device:R
- added R7: 10R 1%, Resistor_SMD:R_0603_1608Metric, symbol Device:R
- added R9: 1k 1%, Resistor_SMD:R_0603_1608Metric, symbol Device:R
- added SW1: SETUP / EVENT / RESET, Button_Switch_SMD:SW_SPST_PTS810, symbol Switch:SW_Push
- added TP1: VBUS, TestPoint:TestPoint_Pad_D1.5mm, symbol Connector:TestPoint
- added TP10: I2C_SCL, TestPoint:TestPoint_Pad_D1.5mm, symbol Connector:TestPoint
- added TP11: USB_DP, TestPoint:TestPoint_Pad_D1.5mm, symbol Connector:TestPoint
- added TP12: USB_DM, TestPoint:TestPoint_Pad_D1.5mm, symbol Connector:TestPoint
- added TP13: CC1_SENSE, TestPoint:TestPoint_Pad_D1.5mm, symbol Connector:TestPoint
- added TP14: CC2_SENSE, TestPoint:TestPoint_Pad_D1.5mm, symbol Connector:TestPoint
- added TP15: PM_ENABLE, TestPoint:TestPoint_Pad_D1.5mm, symbol Connector:TestPoint
- added TP16: USER_BUTTON_N, TestPoint:TestPoint_Pad_D1.5mm, symbol Connector:TestPoint
- added TP17: PM_UART_RX, TestPoint:TestPoint_Pad_D1.5mm, symbol Connector:TestPoint
- added TP18: PM_UART_TX, TestPoint:TestPoint_Pad_D1.5mm, symbol Connector:TestPoint
- added TP19: SGP_VDD, TestPoint:TestPoint_Pad_D1.5mm, symbol Connector:TestPoint
- added TP2: VBUS_FUSED, TestPoint:TestPoint_Pad_D1.5mm, symbol Connector:TestPoint
- added TP3: +3V3, TestPoint:TestPoint_Pad_D1.5mm, symbol Connector:TestPoint
- added TP4: GND, TestPoint:TestPoint_Pad_D1.5mm, symbol Connector:TestPoint
- added TP5: PM_5V, TestPoint:TestPoint_Pad_D1.5mm, symbol Connector:TestPoint
- added TP6: REG_PG, TestPoint:TestPoint_Pad_D1.5mm, symbol Connector:TestPoint
- added TP7: EN, TestPoint:TestPoint_Pad_D1.5mm, symbol Connector:TestPoint
- added TP8: BOOT_GPIO9, TestPoint:TestPoint_Pad_D1.5mm, symbol Connector:TestPoint
- added TP9: I2C_SDA, TestPoint:TestPoint_Pad_D1.5mm, symbol Connector:TestPoint
- added U1: ESP32-C3-WROOM-02-N4, RF_Module:ESP32-C3-WROOM-02, symbol bench-breathe:ESP32-C3-WROOM-02-N4
- added U2: SPS30, symbol bench-breathe:SPS30
- added U3: SGP40-D-R4, bench-breathe:Sensirion_DFN-6-1EP_2.44x2.44mm_P0.8mm, symbol bench-breathe:SGP40-D-R4
- added U4: SHT40-AD1B-R2, Sensor_Humidity:Sensirion_DFN-4_1.5x1.5mm_P0.8mm_SHT4x_NoCentralPad, symbol bench-breathe:SHT40-AD1B-R2
- added U5: TPS62162DSGR, Package_SON:WSON-8-1EP_2x2mm_P0.5mm_EP0.9x1.6mm_ThermalVias, symbol bench-breathe:TPS62162DSGR
- added U6: TPD4E05U06DQAR, Package_SON:USON-10_2.5x1.0mm_P0.5mm, symbol bench-breathe:TPD4E05U06DQAR
- added U7: TPS22919DCKR, Package_TO_SOT_SMD:SOT-363_SC-70-6, symbol bench-breathe:TPS22919DCKR
- D1: footprint (none) -> Diode_SMD:D_SMB; BOM Comments Unidirectional VBUS transient clamp: symbol pin 1 K/cathode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 -> Unidirectional TVS: pin 1 cathode to VBUS_FUSED, pin 2 anod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
- F1: footprint (none) -> Fuse:Fuse_1812_4532Metric; BOM Comments Resettable fault protection, not a precision 500 mA current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 -> Resettable input fault protection; not a precision USB curr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
Connections:
- net VBUS: now reaches F1.1
- net VBUS: now also J1.A4 (VBUS), J1.A9 (VBUS), J1.B4 (VBUS), J1.B9 (VBUS), TP1.1
- net VBUS_FUSED: now reaches F1.2
- net VBUS_FUSED: now also D1.1 (K), C1.1, TP2.1, U5.2 (VIN), U5.3 (EN), U7.1 (IN)
- net GND: now reaches D1.2 (A)
- net GND: now also C1.2, C10.2, C2.2, C3.2, C4.2, C5.2, C6.2, C7.2, C8.2, C9.2, J1.A1 (GND), J1.A12 (GND), J1.B1 (GND), J1.B12 (GND), J1.S1 (SHIELD), J2.5 (Pin_5), J3.2 (Pin_2), R1.2, R2.2, SW1.2, TP4.1, U1.19 (GND), U1.9 (GND), U2.5 (GND), U3.2 (VSS), U3.4 (GND), U3.7 (EP_GND), U4.4 (VSS), U5.1 (PGND), U5.4 (AGND), U5.5 (FB), U5.9 (EP_GND), U6.3 (GND), U6.8 (GND), U7.2 (GND)
- new net +3V3: C2.1, C3.1, C4.1, C7.1, C8.1, J3.1 (Pin_1), L1.2, R10.1, R3.1, R4.1, R5.1, R6.1, R7.1, R8.1, R9.1, TP3.1, U1.1 (3V3), U3.5 (VDDH), U4.3 (VDD), U5.6 (VOS)
- new net BOOT_GPIO9: J3.4 (Pin_4), R10.2, TP8.1, U1.8 (GPIO9)
- new net CC1_SENSE: J1.A5 (CC1), R1.1, TP13.1, U1.18 (GPIO0), U6.4 (D2+)
- new net CC2_SENSE: J1.B5 (CC2), R2.1, TP14.1, U1.17 (GPIO1), U6.5 (D2-)
- new net EN: C5.1, J3.3 (Pin_3), R4.2, TP7.1, U1.2 (EN)
- new net I2C_SCL: R6.2, TP10.1, U1.4 (GPIO5), U3.6 (SCL), U4.2 (SCL)
- new net I2C_SDA: R5.2, TP9.1, U1.3 (GPIO4), U3.3 (SDA), U4.1 (SDA)
- new net PM_5V: C10.1, J2.1 (Pin_1), TP5.1, U2.1 (VDD), U7.5 (QOD), U7.6 (VOUT)
- new net PM_ENABLE: TP15.1, U1.5 (GPIO6), U7.3 (ON)
- new net PM_UART_RX: J2.2 (Pin_2), J3.5 (Pin_5), TP17.1, U1.12 (GPIO21_U0TXD), U2.2 (RX_SDA)
- new net PM_UART_TX: J2.3 (Pin_3), J3.6 (Pin_6), TP18.1, U1.11 (GPIO20_U0RXD), U2.3 (TX_SCL)
- new net REG_PG: R3.2, TP6.1, U1.15 (GPIO3), U5.8 (PG)
- new net SGP_VDD: C6.1, R7.2, TP19.1, U3.1 (VDD)
- new net STATUS_LED_A: D2.2 (A), R9.2
- new net STATUS_LED_K: D2.1 (K), U1.6 (GPIO7)
- new net SW_NODE: L1.1, U5.7 (SW)
- new net USB_CONN_DM: J1.A7 (D-), J1.B7 (D-), R11.1, U6.1 (D1+)
- new net USB_CONN_DP: J1.A6 (D+), J1.B6 (D+), R12.1, U6.2 (D1-)
- new net USB_DM: R11.2, TP12.1, U1.13 (GPIO18_USB_D-)
- new net USB_DP: R12.2, TP11.1, U1.14 (GPIO19_USB_D+)
- new net USER_BUTTON_N: C9.1, R8.2, SW1.1, TP16.1, U1.10 (GPIO10)
- no-connect marks 79 -> 11
Other:
- note added: "LOCAL STATUS + SUSTAINED-ACTION BUTTON"
- note added: "STATIC SCHEMATIC/ERC EVIDENCE ONLY — PCB, SIMULATION, ASSEMBLY, BENCH AND FIELD VALIDATION REMAIN PENDING"
- note added: "SWITCHED SPS30 / SGP40 + SHT40 SHARED I2C"
- note added: "TPS62162 FIXED 3.3 V BUCK / ESP32-C3-WROOM-02 / DEBUG"
- note added: "USB-C 5 V SELV / CC SOURCE SENSE / PPTC / TVS / ESD"
- note removed: "All pins are intentionally marked no-connect so this staging sheet proves editable KiCad metadata without implying a completed circuit."
- note removed: "M2 COMPONENT-SELECTION CARRIER ONLY — NOT AN ELECTRICALLY COMPLETE DESIGN. Issue #3 owns functional wiring, final symbols/footprints, and design ERC."
- company: (none) -> Open hardware design — rwrife/bench-breathe
- title: Bench Breathe M2 Component Selection -> Bench Breathe USB/SELV air-quality trend logger
